File: KiCAD Project/Sydney-live-rail.kicad_pcb (KiCad board)
At the start: 2 copper layers, 255 parts, among them Q1 HL3415A, Q2 MMBT3904, U1 RT9080-33GJ5, U2 ESP32-C3FH4, U3 LTR-303ALS-01, U5 SN74LV1T34DBV

Commit message: Added annotations to schematic
Parts:
- removed C1, C100, C101, C102, C103, C104, C105, C106, C107, C108, C109, C11, C110, C111, C112, C113, C114, C115, C116, C117, C118, C119, C12, C120, C121, C122, C123, C13, C14, C16, C2, C3, C35, C4, C6, C7, C8, C9: 10uF, PCM_JLCPCB:C_0402
- removed C15, C17, C18, C5: 47uF, PCM_JLCPCB:C_0805
- removed C19, C20: 27pF, PCM_JLCPCB:C_0402
- removed C36, C37: 1.5pF, PCM_JLCPCB:C_0402
- removed D1: MMSZ5227B, PCM_JLCPCB:D_SOD-123
- removed D10, D11, D2: Red, PCM_JLCPCB:D_0805
- removed D100, D101, D102, D103, D104, D105, D106, D107, D108, D109, D110, D111, D112, D113, D114, D115, D116, D117, D118, D119, D120, D121, D122, D123, D124, D125, D126, D127, D128, D129, D130, D131, D132, D133, D134, D135, D136, D137, D138, D139, D140, D141, D142, D143, D144, D145, D146, D147, D148, D149, D150, D151, D152, D153, D154, D155, D156, D157, D158, D159, D160, D161, D162, D163, D164, D165, D166, D167, D168, D169, D170, D171, D172, D173, D174, D175, D176, D177, D178, D179, D180, D181, D182, D183, D184, D185, D186, D187, D188, D189, D190, D191, D192, D193, D194, D195, D196, D197, D198, D199, D200, D201, D202, D203, D204, D205, D206, D207, D208, D209, D210, D211, D212, D213, D214, D215, D216, D217, D218, D219, D220, D221, D222, D223, D224, D225, D226, D227, D228, D229, D230, D231, D232, D233, D234, D235, D236, D237, D238, D239, D240, D241, D242, D243, D244, D245, D246, D247, D248, D249, D250, D251, D252, D253, D254, D255, D256, D257, D258, D259, D260, D261, D262, D263, D264, D265, D266: XL-1615RGBC-WS2812B-S, PCM_JLCPCB:LED-SMD_4P-L1.6-W1.5_XL-1615RGBC-WS2812B
- removed D12, D8, D9: Green, PCM_JLCPCB:D_0805
- removed D13: H3V3U10B, PCM_JLCPCB:D_DFN1006-2L
- removed D4, D5: MM1W5V6, PCM_JLCPCB:D_SOD-123
- removed F1: Polyfuse, 2A, Fuse:Fuse_1206_3216Metric
- removed L1: 2.7nH, PCM_JLCPCB:L_0402
- removed L5: 15nH,300mA, PCM_JLCPCB:L_0402
- removed Q1: HL3415A, PCM_JLCPCB:Q_SOT-23
- removed Q2: MMBT3904, PCM_JLCPCB:Q_SOT-23
- removed R1, R12, R17, R2, R21, R3, R5, R8: 10kΩ, PCM_JLCPCB:R_0402
- removed R13, R14, R4: 5.1kΩ, PCM_JLCPCB:R_0402
- removed R15, R18, R7: 510Ω, PCM_JLCPCB:R_0402
- removed R16, R22, R23, R25, R9: 100kΩ, PCM_JLCPCB:R_0402
- removed S1, S2, S3, S4: Tactile Button, 160gf, PCM_JLCPCB:SW-SMD_4P-L5.1-W5.1-P3.70-LS6.5-TL-2
- removed U1: RT9080-33GJ5, Package_TO_SOT_SMD:TSOT-23-5
- removed U2: ESP32-C3FH4, PCM_JLCPCB:QFN-32-1EP_5x5mm_P0.5mm_EP3.7x3.7mm_ThermalVias
- removed U3: LTR-303ALS-01, PCM_JLCPCB:Lite-On_LTR-303ALS-01
- removed U5: SN74LV1T34DBV, Package_TO_SOT_SMD:SOT-23-5

Commit message: Added control electronics from Wellington project
Parts:
- added AE1: Antenna_Shield, Custom_Footprints:Inverted_F_Antenna_2.4Ghz_1.0mmPCB_TI_CC2430DB.pretty, F.Cu at (49.1, 355.3)
- added C1: 10uF, PCM_JLCPCB:C_0402, F.Cu at (62.5, 357.0)
- added C100: 10uF, PCM_JLCPCB:C_0402, F.Cu at (179.2, -169.6)
- added C101: 10uF, PCM_JLCPCB:C_0402, F.Cu at (179.2, -167.8)
- added C102: 10uF, PCM_JLCPCB:C_0402, F.Cu at (179.2, -165.9)
- added C103: 10uF, PCM_JLCPCB:C_0402, F.Cu at (179.2, -164.1)
- added C104: 10uF, PCM_JLCPCB:C_0402, F.Cu at (179.2, -162.2)
- added C105: 10uF, PCM_JLCPCB:C_0402, F.Cu at (179.2, -160.3)
- added C106: 10uF, PCM_JLCPCB:C_0402, F.Cu at (182.1, -169.6)
- added C107: 10uF, PCM_JLCPCB:C_0402, F.Cu at (182.1, -167.8)
- added C108: 10uF, PCM_JLCPCB:C_0402, F.Cu at (182.1, -165.9)
- added C109: 10uF, PCM_JLCPCB:C_0402, F.Cu at (182.1, -164.1)
- added C11: 10uF, PCM_JLCPCB:C_0402, F.Cu at (76.4, 352.0)
- added C110: 10uF, PCM_JLCPCB:C_0402, F.Cu at (182.1, -162.2)
- added C111: 10uF, PCM_JLCPCB:C_0402, F.Cu at (182.1, -160.3)
- added C112: 10uF, PCM_JLCPCB:C_0402, F.Cu at (184.9, -169.6)
- added C113: 10uF, PCM_JLCPCB:C_0402, F.Cu at (184.9, -167.8)
- added C114: 10uF, PCM_JLCPCB:C_0402, F.Cu at (184.9, -165.9)
- added C115: 10uF, PCM_JLCPCB:C_0402, F.Cu at (184.9, -164.1)
- added C116: 10uF, PCM_JLCPCB:C_0402, F.Cu at (184.9, -162.2)
- added C117: 10uF, PCM_JLCPCB:C_0402, F.Cu at (184.9, -160.3)
- added C118: 10uF, PCM_JLCPCB:C_0402, F.Cu at (187.8, -169.6)
- added C119: 10uF, PCM_JLCPCB:C_0402, F.Cu at (187.8, -167.8)
- added C12: 10uF, PCM_JLCPCB:C_0402, F.Cu at (75.7, 351.3)
- added C120: 10uF, PCM_JLCPCB:C_0402, F.Cu at (187.8, -165.9)
- added C121: 10uF, PCM_JLCPCB:C_0402, F.Cu at (187.8, -164.1)
- added C122: 10uF, PCM_JLCPCB:C_0402, F.Cu at (187.8, -162.2)
- added C123: 10uF, PCM_JLCPCB:C_0402, F.Cu at (187.8, -160.3)
- added C13: 10uF, PCM_JLCPCB:C_0402, F.Cu at (133.5, 353.1)
- added C14: 10uF, PCM_JLCPCB:C_0402, F.Cu at (68.8, 353.5)
- added C15: 47uF, PCM_JLCPCB:C_0805, F.Cu at (60.9, 347.9)
- added C16: 10uF, PCM_JLCPCB:C_0402, F.Cu at (72.9, 357.6)
- added C17: 47uF, PCM_JLCPCB:C_0805, F.Cu at (65.8, 357.5)
- added C18: 47uF, PCM_JLCPCB:C_0805, F.Cu at (105.0, 355.8)
- added C19: 27pF, PCM_JLCPCB:C_0402, F.Cu at (62.1, 337.2)
- added C2: 10uF, PCM_JLCPCB:C_0402, F.Cu at (100.8, 359.0)
- added C20: 27pF, PCM_JLCPCB:C_0402, F.Cu at (59.3, 341.1)
- added C3: 10uF, PCM_JLCPCB:C_0402, F.Cu at (62.5, 352.1)
- added C35: 10uF, PCM_JLCPCB:C_0402, F.Cu at (94.3, 355.9)
- added C36: 1.5pF, PCM_JLCPCB:C_0402, F.Cu at (60.5, 343.9)
- added C37: 1.5pF, PCM_JLCPCB:C_0402, F.Cu at (57.9, 344.9)
- added C4: 10uF, PCM_JLCPCB:C_0402, F.Cu at (61.5, 346.0)
- added C5: 47uF, PCM_JLCPCB:C_0805, F.Cu at (60.9, 349.9)
- added C6: 10uF, PCM_JLCPCB:C_0402, F.Cu at (68.5, 341.9)
- added C7: 10uF, PCM_JLCPCB:C_0402, F.Cu at (61.1, 342.5)
- added C8: 10uF, PCM_JLCPCB:C_0402, F.Cu at (69.1, 342.5)
- added C9: 10uF, PCM_JLCPCB:C_0402, F.Cu at (67.6, 347.6)
- added D1: MMSZ5227B, PCM_JLCPCB:D_SOD-123, F.Cu at (59.8, 354.5)
- added D10: Red, PCM_JLCPCB:D_0805, F.Cu at (63.3, 363.0)
- added D100: XL-1615RGBC-WS2812B-S, PCM_JLCPCB:LED-SMD_4P-L1.6-W1.5_XL-1615RGBC-WS2812B, F.Cu at (101.3, 67.0)
- added D101: XL-1615RGBC-WS2812B-S, PCM_JLCPCB:LED-SMD_4P-L1.6-W1.5_XL-1615RGBC-WS2812B, F.Cu at (98.0, 66.6)
- added D102: XL-1615RGBC-WS2812B-S, PCM_JLCPCB:LED-SMD_4P-L1.6-W1.5_XL-1615RGBC-WS2812B, F.Cu at (94.8, 66.3)
- added D103: XL-1615RGBC-WS2812B-S, PCM_JLCPCB:LED-SMD_4P-L1.6-W1.5_XL-1615RGBC-WS2812B, F.Cu at (93.0, 69.0)
- added D104: XL-1615RGBC-WS2812B-S, PCM_JLCPCB:LED-SMD_4P-L1.6-W1.5_XL-1615RGBC-WS2812B, F.Cu at (91.8, 72.1)
- added D105: XL-1615RGBC-WS2812B-S, PCM_JLCPCB:LED-SMD_4P-L1.6-W1.5_XL-1615RGBC-WS2812B, F.Cu at (91.6, 75.4)
- added D106: XL-1615RGBC-WS2812B-S, PCM_JLCPCB:LED-SMD_4P-L1.6-W1.5_XL-1615RGBC-WS2812B, F.Cu at (91.4, 78.7)
- added D107: XL-1615RGBC-WS2812B-S, PCM_JLCPCB:LED-SMD_4P-L1.6-W1.5_XL-1615RGBC-WS2812B, F.Cu at (91.0, 82.5)
- added D108: XL-1615RGBC-WS2812B-S, PCM_JLCPCB:LED-SMD_4P-L1.6-W1.5_XL-1615RGBC-WS2812B, F.Cu at (90.7, 86.3)
- added D109: XL-1615RGBC-WS2812B-S, PCM_JLCPCB:LED-SMD_4P-L1.6-W1.5_XL-1615RGBC-WS2812B, F.Cu at (90.3, 90.1)
- added D11: Red, PCM_JLCPCB:D_0805, F.Cu at (75.7, 363.0)
- added D110: XL-1615RGBC-WS2812B-S, PCM_JLCPCB:LED-SMD_4P-L1.6-W1.5_XL-1615RGBC-WS2812B, F.Cu at (90.0, 93.3)
- added D111: XL-1615RGBC-WS2812B-S, PCM_JLCPCB:LED-SMD_4P-L1.6-W1.5_XL-1615RGBC-WS2812B, F.Cu at (89.7, 96.5)
- added D112: XL-1615RGBC-WS2812B-S, PCM_JLCPCB:LED-SMD_4P-L1.6-W1.5_XL-1615RGBC-WS2812B, F.Cu at (89.5, 99.7)
- added D113: XL-1615RGBC-WS2812B-S, PCM_JLCPCB:LED-SMD_4P-L1.6-W1.5_XL-1615RGBC-WS2812B, F.Cu at (89.5, 102.9)
- added D114: XL-1615RGBC-WS2812B-S, PCM_JLCPCB:LED-SMD_4P-L1.6-W1.5_XL-1615RGBC-WS2812B, F.Cu at (89.5, 106.1)
- added D115: XL-1615RGBC-WS2812B-S, PCM_JLCPCB:LED-SMD_4P-L1.6-W1.5_XL-1615RGBC-WS2812B, F.Cu at (89.5, 109.3)
- added D116: XL-1615RGBC-WS2812B-S, PCM_JLCPCB:LED-SMD_4P-L1.6-W1.5_XL-1615RGBC-WS2812B, F.Cu at (89.6, 112.5)
- added D117: XL-1615RGBC-WS2812B-S, PCM_JLCPCB:LED-SMD_4P-L1.6-W1.5_XL-1615RGBC-WS2812B, F.Cu at (89.7, 115.7)
- added D118: XL-1615RGBC-WS2812B-S, PCM_JLCPCB:LED-SMD_4P-L1.6-W1.5_XL-1615RGBC-WS2812B, F.Cu at (89.6, 118.9)
- added D119: XL-1615RGBC-WS2812B-S, PCM_JLCPCB:LED-SMD_4P-L1.6-W1.5_XL-1615RGBC-WS2812B, F.Cu at (89.3, 122.1)
- added D12: Green, PCM_JLCPCB:D_0805, F.Cu at (75.7, 365.0)
- added D120: XL-1615RGBC-WS2812B-S, PCM_JLCPCB:LED-SMD_4P-L1.6-W1.5_XL-1615RGBC-WS2812B, F.Cu at (88.9, 125.0)
- added D121: XL-1615RGBC-WS2812B-S, PCM_JLCPCB:LED-SMD_4P-L1.6-W1.5_XL-1615RGBC-WS2812B, F.Cu at (88.1, 128.0)
- added D122: XL-1615RGBC-WS2812B-S, PCM_JLCPCB:LED-SMD_4P-L1.6-W1.5_XL-1615RGBC-WS2812B, F.Cu at (87.2, 130.9)
- added D123: XL-1615RGBC-WS2812B-S, PCM_JLCPCB:LED-SMD_4P-L1.6-W1.5_XL-1615RGBC-WS2812B, F.Cu at (86.4, 133.8)
- added D124: XL-1615RGBC-WS2812B-S, PCM_JLCPCB:LED-SMD_4P-L1.6-W1.5_XL-1615RGBC-WS2812B, F.Cu at (85.7, 136.7)
- added D125: XL-1615RGBC-WS2812B-S, PCM_JLCPCB:LED-SMD_4P-L1.6-W1.5_XL-1615RGBC-WS2812B, F.Cu at (84.9, 139.6)
- added D126: XL-1615RGBC-WS2812B-S, PCM_JLCPCB:LED-SMD_4P-L1.6-W1.5_XL-1615RGBC-WS2812B, F.Cu at (84.4, 142.6)
- added D127: XL-1615RGBC-WS2812B-S, PCM_JLCPCB:LED-SMD_4P-L1.6-W1.5_XL-1615RGBC-WS2812B, F.Cu at (83.8, 146.1)
- added D128: XL-1615RGBC-WS2812B-S, PCM_JLCPCB:LED-SMD_4P-L1.6-W1.5_XL-1615RGBC-WS2812B, F.Cu at (82.8, 149.5)
- added D129: XL-1615RGBC-WS2812B-S, PCM_JLCPCB:LED-SMD_4P-L1.6-W1.5_XL-1615RGBC-WS2812B, F.Cu at (81.9, 152.8)
- added D13: H3V3U10B, PCM_JLCPCB:D_DFN1006-2L, F.Cu at (57.0, 344.0)
- added D130: XL-1615RGBC-WS2812B-S, PCM_JLCPCB:LED-SMD_4P-L1.6-W1.5_XL-1615RGBC-WS2812B, F.Cu at (83.6, 155.5)
- added D131: XL-1615RGBC-WS2812B-S, PCM_JLCPCB:LED-SMD_4P-L1.6-W1.5_XL-1615RGBC-WS2812B, F.Cu at (86.0, 157.2)
- added D132: XL-1615RGBC-WS2812B-S, PCM_JLCPCB:LED-SMD_4P-L1.6-W1.5_XL-1615RGBC-WS2812B, F.Cu at (88.5, 158.9)
- added D133: XL-1615RGBC-WS2812B-S, PCM_JLCPCB:LED-SMD_4P-L1.6-W1.5_XL-1615RGBC-WS2812B, F.Cu at (91.0, 160.5)
- added D134: XL-1615RGBC-WS2812B-S, PCM_JLCPCB:LED-SMD_4P-L1.6-W1.5_XL-1615RGBC-WS2812B, F.Cu at (93.5, 162.2)
- added D135: XL-1615RGBC-WS2812B-S, PCM_JLCPCB:LED-SMD_4P-L1.6-W1.5_XL-1615RGBC-WS2812B, F.Cu at (93.7, 165.1)
- added D136: XL-1615RGBC-WS2812B-S, PCM_JLCPCB:LED-SMD_4P-L1.6-W1.5_XL-1615RGBC-WS2812B, F.Cu at (92.1, 167.6)
- added D137: XL-1615RGBC-WS2812B-S, PCM_JLCPCB:LED-SMD_4P-L1.6-W1.5_XL-1615RGBC-WS2812B, F.Cu at (90.4, 170.2)
- added D138: XL-1615RGBC-WS2812B-S, PCM_JLCPCB:LED-SMD_4P-L1.6-W1.5_XL-1615RGBC-WS2812B, F.Cu at (89.5, 173.1)
- added D139: XL-1615RGBC-WS2812B-S, PCM_JLCPCB:LED-SMD_4P-L1.6-W1.5_XL-1615RGBC-WS2812B, F.Cu at (91.2, 175.5)
- added D140: XL-1615RGBC-WS2812B-S, PCM_JLCPCB:LED-SMD_4P-L1.6-W1.5_XL-1615RGBC-WS2812B, F.Cu at (93.8, 177.3)
- added D141: XL-1615RGBC-WS2812B-S, PCM_JLCPCB:LED-SMD_4P-L1.6-W1.5_XL-1615RGBC-WS2812B, F.Cu at (96.3, 179.1)
- added D142: XL-1615RGBC-WS2812B-S, PCM_JLCPCB:LED-SMD_4P-L1.6-W1.5_XL-1615RGBC-WS2812B, F.Cu at (99.1, 180.4)
- added D143: XL-1615RGBC-WS2812B-S, PCM_JLCPCB:LED-SMD_4P-L1.6-W1.5_XL-1615RGBC-WS2812B, F.Cu at (101.9, 181.8)
- added D144: XL-1615RGBC-WS2812B-S, PCM_JLCPCB:LED-SMD_4P-L1.6-W1.5_XL-1615RGBC-WS2812B, F.Cu at (104.7, 183.2)
- added D145: XL-1615RGBC-WS2812B-S, PCM_JLCPCB:LED-SMD_4P-L1.6-W1.5_XL-1615RGBC-WS2812B, F.Cu at (107.4, 184.8)
- added D146: XL-1615RGBC-WS2812B-S, PCM_JLCPCB:LED-SMD_4P-L1.6-W1.5_XL-1615RGBC-WS2812B, F.Cu at (110.1, 186.3)
- added D147: XL-1615RGBC-WS2812B-S, PCM_JLCPCB:LED-SMD_4P-L1.6-W1.5_XL-1615RGBC-WS2812B, F.Cu at (112.7, 188.0)
- added D148: XL-1615RGBC-WS2812B-S, PCM_JLCPCB:LED-SMD_4P-L1.6-W1.5_XL-1615RGBC-WS2812B, F.Cu at (115.4, 189.6)
- added D149: XL-1615RGBC-WS2812B-S, PCM_JLCPCB:LED-SMD_4P-L1.6-W1.5_XL-1615RGBC-WS2812B, F.Cu at (118.1, 191.0)
- added D150: XL-1615RGBC-WS2812B-S, PCM_JLCPCB:LED-SMD_4P-L1.6-W1.5_XL-1615RGBC-WS2812B, F.Cu at (121.0, 192.0)
- added D151: XL-1615RGBC-WS2812B-S, PCM_JLCPCB:LED-SMD_4P-L1.6-W1.5_XL-1615RGBC-WS2812B, F.Cu at (124.1, 192.4)
- added D152: XL-1615RGBC-WS2812B-S, PCM_JLCPCB:LED-SMD_4P-L1.6-W1.5_XL-1615RGBC-WS2812B, F.Cu at (127.1, 192.9)
- added D153: XL-1615RGBC-WS2812B-S, PCM_JLCPCB:LED-SMD_4P-L1.6-W1.5_XL-1615RGBC-WS2812B, F.Cu at (130.2, 193.4)
- added D154: XL-1615RGBC-WS2812B-S, PCM_JLCPCB:LED-SMD_4P-L1.6-W1.5_XL-1615RGBC-WS2812B, F.Cu at (133.2, 193.9)
- added D155: XL-1615RGBC-WS2812B-S, PCM_JLCPCB:LED-SMD_4P-L1.6-W1.5_XL-1615RGBC-WS2812B, F.Cu at (136.2, 194.7)
- added D156: XL-1615RGBC-WS2812B-S, PCM_JLCPCB:LED-SMD_4P-L1.6-W1.5_XL-1615RGBC-WS2812B, F.Cu at (138.8, 196.3)
- added D157: XL-1615RGBC-WS2812B-S, PCM_JLCPCB:LED-SMD_4P-L1.6-W1.5_XL-1615RGBC-WS2812B, F.Cu at (141.4, 198.0)
- added D158: XL-1615RGBC-WS2812B-S, PCM_JLCPCB:LED-SMD_4P-L1.6-W1.5_XL-1615RGBC-WS2812B, F.Cu at (142.8, 200.6)
- added D159: XL-1615RGBC-WS2812B-S, PCM_JLCPCB:LED-SMD_4P-L1.6-W1.5_XL-1615RGBC-WS2812B, F.Cu at (143.4, 203.7)
- added D160: XL-1615RGBC-WS2812B-S, PCM_JLCPCB:LED-SMD_4P-L1.6-W1.5_XL-1615RGBC-WS2812B, F.Cu at (143.9, 206.7)
- added D161: XL-1615RGBC-WS2812B-S, PCM_JLCPCB:LED-SMD_4P-L1.6-W1.5_XL-1615RGBC-WS2812B, F.Cu at (144.4, 209.7)
- added D162: XL-1615RGBC-WS2812B-S, PCM_JLCPCB:LED-SMD_4P-L1.6-W1.5_XL-1615RGBC-WS2812B, F.Cu at (144.8, 212.8)
- added D163: XL-1615RGBC-WS2812B-S, PCM_JLCPCB:LED-SMD_4P-L1.6-W1.5_XL-1615RGBC-WS2812B, F.Cu at (145.2, 215.9)
- added D164: XL-1615RGBC-WS2812B-S, PCM_JLCPCB:LED-SMD_4P-L1.6-W1.5_XL-1615RGBC-WS2812B, F.Cu at (145.5, 219.0)
- added D165: XL-1615RGBC-WS2812B-S, PCM_JLCPCB:LED-SMD_4P-L1.6-W1.5_XL-1615RGBC-WS2812B, F.Cu at (146.0, 222.0)
- added D166: XL-1615RGBC-WS2812B-S, PCM_JLCPCB:LED-SMD_4P-L1.6-W1.5_XL-1615RGBC-WS2812B, F.Cu at (146.4, 225.1)
- added D167: XL-1615RGBC-WS2812B-S, PCM_JLCPCB:LED-SMD_4P-L1.6-W1.5_XL-1615RGBC-WS2812B, F.Cu at (146.9, 228.2)
- added D168: XL-1615RGBC-WS2812B-S, PCM_JLCPCB:LED-SMD_4P-L1.6-W1.5_XL-1615RGBC-WS2812B, F.Cu at (147.3, 231.3)
- added D169: XL-1615RGBC-WS2812B-S, PCM_JLCPCB:LED-SMD_4P-L1.6-W1.5_XL-1615RGBC-WS2812B, F.Cu at (147.7, 234.3)
- added D170: XL-1615RGBC-WS2812B-S, PCM_JLCPCB:LED-SMD_4P-L1.6-W1.5_XL-1615RGBC-WS2812B, F.Cu at (148.1, 237.4)
- added D171: XL-1615RGBC-WS2812B-S, PCM_JLCPCB:LED-SMD_4P-L1.6-W1.5_XL-1615RGBC-WS2812B, F.Cu at (148.4, 240.5)
- added D172: XL-1615RGBC-WS2812B-S, PCM_JLCPCB:LED-SMD_4P-L1.6-W1.5_XL-1615RGBC-WS2812B, F.Cu at (149.2, 243.5)
- added D173: XL-1615RGBC-WS2812B-S, PCM_JLCPCB:LED-SMD_4P-L1.6-W1.5_XL-1615RGBC-WS2812B, F.Cu at (151.1, 245.9)
- added D174: XL-1615RGBC-WS2812B-S, PCM_JLCPCB:LED-SMD_4P-L1.6-W1.5_XL-1615RGBC-WS2812B, F.Cu at (153.2, 248.2)
- added D175: XL-1615RGBC-WS2812B-S, PCM_JLCPCB:LED-SMD_4P-L1.6-W1.5_XL-1615RGBC-WS2812B, F.Cu at (155.4, 250.4)
- added D176: XL-1615RGBC-WS2812B-S, PCM_JLCPCB:LED-SMD_4P-L1.6-W1.5_XL-1615RGBC-WS2812B, F.Cu at (157.6, 252.5)
- added D177: XL-1615RGBC-WS2812B-S, PCM_JLCPCB:LED-SMD_4P-L1.6-W1.5_XL-1615RGBC-WS2812B, F.Cu at (160.0, 254.5)
- added D178: XL-1615RGBC-WS2812B-S, PCM_JLCPCB:LED-SMD_4P-L1.6-W1.5_XL-1615RGBC-WS2812B, F.Cu at (162.7, 255.9)
- added D179: XL-1615RGBC-WS2812B-S, PCM_JLCPCB:LED-SMD_4P-L1.6-W1.5_XL-1615RGBC-WS2812B, F.Cu at (165.3, 257.8)
- added D180: XL-1615RGBC-WS2812B-S, PCM_JLCPCB:LED-SMD_4P-L1.6-W1.5_XL-1615RGBC-WS2812B, F.Cu at (167.8, 259.4)
- added D181: XL-1615RGBC-WS2812B-S, PCM_JLCPCB:LED-SMD_4P-L1.6-W1.5_XL-1615RGBC-WS2812B, F.Cu at (170.7, 260.8)
- added D182: XL-1615RGBC-WS2812B-S, PCM_JLCPCB:LED-SMD_4P-L1.6-W1.5_XL-1615RGBC-WS2812B, F.Cu at (173.5, 262.1)
- added D183: XL-1615RGBC-WS2812B-S, PCM_JLCPCB:LED-SMD_4P-L1.6-W1.5_XL-1615RGBC-WS2812B, F.Cu at (176.4, 263.5)
- added D184: XL-1615RGBC-WS2812B-S, PCM_JLCPCB:LED-SMD_4P-L1.6-W1.5_XL-1615RGBC-WS2812B, F.Cu at (178.6, 265.5)
- added D185: XL-1615RGBC-WS2812B-S, PCM_JLCPCB:LED-SMD_4P-L1.6-W1.5_XL-1615RGBC-WS2812B, F.Cu at (180.7, 267.6)
- added D186: XL-1615RGBC-WS2812B-S, PCM_JLCPCB:LED-SMD_4P-L1.6-W1.5_XL-1615RGBC-WS2812B, F.Cu at (183.4, 269.3)
- added D187: XL-1615RGBC-WS2812B-S, PCM_JLCPCB:LED-SMD_4P-L1.6-W1.5_XL-1615RGBC-WS2812B, F.Cu at (186.1, 271.0)
- added D188: XL-1615RGBC-WS2812B-S, PCM_JLCPCB:LED-SMD_4P-L1.6-W1.5_XL-1615RGBC-WS2812B, F.Cu at (188.3, 273.2)
- added D189: XL-1615RGBC-WS2812B-S, PCM_JLCPCB:LED-SMD_4P-L1.6-W1.5_XL-1615RGBC-WS2812B, F.Cu at (189.9, 275.9)
- added D190: XL-1615RGBC-WS2812B-S, PCM_JLCPCB:LED-SMD_4P-L1.6-W1.5_XL-1615RGBC-WS2812B, F.Cu at (191.2, 278.8)
- added D191: XL-1615RGBC-WS2812B-S, PCM_JLCPCB:LED-SMD_4P-L1.6-W1.5_XL-1615RGBC-WS2812B, F.Cu at (192.4, 281.7)
- added D192: XL-1615RGBC-WS2812B-S, PCM_JLCPCB:LED-SMD_4P-L1.6-W1.5_XL-1615RGBC-WS2812B, F.Cu at (194.1, 284.4)
- added D193: XL-1615RGBC-WS2812B-S, PCM_JLCPCB:LED-SMD_4P-L1.6-W1.5_XL-1615RGBC-WS2812B, F.Cu at (195.6, 287.2)
- added D194: XL-1615RGBC-WS2812B-S, PCM_JLCPCB:LED-SMD_4P-L1.6-W1.5_XL-1615RGBC-WS2812B, F.Cu at (195.1, 290.3)
- added D195: XL-1615RGBC-WS2812B-S, PCM_JLCPCB:LED-SMD_4P-L1.6-W1.5_XL-1615RGBC-WS2812B, F.Cu at (194.7, 293.5)
- added D196: XL-1615RGBC-WS2812B-S, PCM_JLCPCB:LED-SMD_4P-L1.6-W1.5_XL-1615RGBC-WS2812B, F.Cu at (194.2, 296.7)
- added D197: XL-1615RGBC-WS2812B-S, PCM_JLCPCB:LED-SMD_4P-L1.6-W1.5_XL-1615RGBC-WS2812B, F.Cu at (193.7, 299.9)
- added D198: XL-1615RGBC-WS2812B-S, PCM_JLCPCB:LED-SMD_4P-L1.6-W1.5_XL-1615RGBC-WS2812B, F.Cu at (193.2, 303.0)
- added D199: XL-1615RGBC-WS2812B-S, PCM_JLCPCB:LED-SMD_4P-L1.6-W1.5_XL-1615RGBC-WS2812B, F.Cu at (192.7, 306.2)
- added D2: Red, PCM_JLCPCB:D_0805, F.Cu at (87.4, 363.0)
- added D200: XL-1615RGBC-WS2812B-S, PCM_JLCPCB:LED-SMD_4P-L1.6-W1.5_XL-1615RGBC-WS2812B, F.Cu at (192.4, 309.3)
- added D201: XL-1615RGBC-WS2812B-S, PCM_JLCPCB:LED-SMD_4P-L1.6-W1.5_XL-1615RGBC-WS2812B, F.Cu at (195.3, 310.4)
- added D202: XL-1615RGBC-WS2812B-S, PCM_JLCPCB:LED-SMD_4P-L1.6-W1.5_XL-1615RGBC-WS2812B, F.Cu at (198.4, 310.9)
- added D203: XL-1615RGBC-WS2812B-S, PCM_JLCPCB:LED-SMD_4P-L1.6-W1.5_XL-1615RGBC-WS2812B, F.Cu at (201.5, 311.5)
- added D204: XL-1615RGBC-WS2812B-S, PCM_JLCPCB:LED-SMD_4P-L1.6-W1.5_XL-1615RGBC-WS2812B, F.Cu at (204.6, 312.0)
- added D205: XL-1615RGBC-WS2812B-S, PCM_JLCPCB:LED-SMD_4P-L1.6-W1.5_XL-1615RGBC-WS2812B, F.Cu at (207.7, 312.6)
- added D206: XL-1615RGBC-WS2812B-S, PCM_JLCPCB:LED-SMD_4P-L1.6-W1.5_XL-1615RGBC-WS2812B, F.Cu at (210.8, 313.1)
- added D207: XL-1615RGBC-WS2812B-S, PCM_JLCPCB:LED-SMD_4P-L1.6-W1.5_XL-1615RGBC-WS2812B, F.Cu at (213.9, 313.7)
- added D208: XL-1615RGBC-WS2812B-S, PCM_JLCPCB:LED-SMD_4P-L1.6-W1.5_XL-1615RGBC-WS2812B, F.Cu at (152.3, 263.6)
- added D209: XL-1615RGBC-WS2812B-S, PCM_JLCPCB:LED-SMD_4P-L1.6-W1.5_XL-1615RGBC-WS2812B, F.Cu at (151.9, 266.8)
- added D210: XL-1615RGBC-WS2812B-S, PCM_JLCPCB:LED-SMD_4P-L1.6-W1.5_XL-1615RGBC-WS2812B, F.Cu at (151.5, 269.9)
- added D211: XL-1615RGBC-WS2812B-S, PCM_JLCPCB:LED-SMD_4P-L1.6-W1.5_XL-1615RGBC-WS2812B, F.Cu at (151.0, 273.0)
- added D212: XL-1615RGBC-WS2812B-S, PCM_JLCPCB:LED-SMD_4P-L1.6-W1.5_XL-1615RGBC-WS2812B, F.Cu at (150.6, 276.2)
- added D213: XL-1615RGBC-WS2812B-S, PCM_JLCPCB:LED-SMD_4P-L1.6-W1.5_XL-1615RGBC-WS2812B, F.Cu at (150.2, 279.3)
- added D214: XL-1615RGBC-WS2812B-S, PCM_JLCPCB:LED-SMD_4P-L1.6-W1.5_XL-1615RGBC-WS2812B, F.Cu at (149.9, 282.5)
- added D215: XL-1615RGBC-WS2812B-S, PCM_JLCPCB:LED-SMD_4P-L1.6-W1.5_XL-1615RGBC-WS2812B, F.Cu at (149.6, 285.7)
- added D216: XL-1615RGBC-WS2812B-S, PCM_JLCPCB:LED-SMD_4P-L1.6-W1.5_XL-1615RGBC-WS2812B, F.Cu at (149.7, 288.9)
- added D217: XL-1615RGBC-WS2812B-S, PCM_JLCPCB:LED-SMD_4P-L1.6-W1.5_XL-1615RGBC-WS2812B, F.Cu at (151.2, 291.7)
- added D218: XL-1615RGBC-WS2812B-S, PCM_JLCPCB:LED-SMD_4P-L1.6-W1.5_XL-1615RGBC-WS2812B, F.Cu at (153.4, 294.0)
- added D219: XL-1615RGBC-WS2812B-S, PCM_JLCPCB:LED-SMD_4P-L1.6-W1.5_XL-1615RGBC-WS2812B, F.Cu at (155.5, 296.4)
- added D220: XL-1615RGBC-WS2812B-S, PCM_JLCPCB:LED-SMD_4P-L1.6-W1.5_XL-1615RGBC-WS2812B, F.Cu at (157.3, 299.0)
- added D221: XL-1615RGBC-WS2812B-S, PCM_JLCPCB:LED-SMD_4P-L1.6-W1.5_XL-1615RGBC-WS2812B, F.Cu at (157.9, 302.1)
- added D222: XL-1615RGBC-WS2812B-S, PCM_JLCPCB:LED-SMD_4P-L1.6-W1.5_XL-1615RGBC-WS2812B, F.Cu at (158.4, 305.3)
- added D223: XL-1615RGBC-WS2812B-S, PCM_JLCPCB:LED-SMD_4P-L1.6-W1.5_XL-1615RGBC-WS2812B, F.Cu at (159.0, 308.4)
- added D224: XL-1615RGBC-WS2812B-S, PCM_JLCPCB:LED-SMD_4P-L1.6-W1.5_XL-1615RGBC-WS2812B, F.Cu at (159.6, 311.6)
- added D225: XL-1615RGBC-WS2812B-S, PCM_JLCPCB:LED-SMD_4P-L1.6-W1.5_XL-1615RGBC-WS2812B, F.Cu at (160.3, 314.8)
- added D226: XL-1615RGBC-WS2812B-S, PCM_JLCPCB:LED-SMD_4P-L1.6-W1.5_XL-1615RGBC-WS2812B, F.Cu at (160.8, 318.1)
- added D227: XL-1615RGBC-WS2812B-S, PCM_JLCPCB:LED-SMD_4P-L1.6-W1.5_XL-1615RGBC-WS2812B, F.Cu at (161.3, 321.4)
- added D228: XL-1615RGBC-WS2812B-S, PCM_JLCPCB:LED-SMD_4P-L1.6-W1.5_XL-1615RGBC-WS2812B, F.Cu at (161.8, 324.7)
- added D229: XL-1615RGBC-WS2812B-S, PCM_JLCPCB:LED-SMD_4P-L1.6-W1.5_XL-1615RGBC-WS2812B, F.Cu at (162.3, 328.0)
- added D230: XL-1615RGBC-WS2812B-S, PCM_JLCPCB:LED-SMD_4P-L1.6-W1.5_XL-1615RGBC-WS2812B, F.Cu at (162.8, 331.3)
- added D231: XL-1615RGBC-WS2812B-S, PCM_JLCPCB:LED-SMD_4P-L1.6-W1.5_XL-1615RGBC-WS2812B, F.Cu at (163.2, 334.6)
- added D232: XL-1615RGBC-WS2812B-S, PCM_JLCPCB:LED-SMD_4P-L1.6-W1.5_XL-1615RGBC-WS2812B, F.Cu at (163.9, 338.1)
- added D233: XL-1615RGBC-WS2812B-S, PCM_JLCPCB:LED-SMD_4P-L1.6-W1.5_XL-1615RGBC-WS2812B, F.Cu at (165.3, 341.2)
- added D234: XL-1615RGBC-WS2812B-S, PCM_JLCPCB:LED-SMD_4P-L1.6-W1.5_XL-1615RGBC-WS2812B, F.Cu at (166.7, 344.4)
- added D235: XL-1615RGBC-WS2812B-S, PCM_JLCPCB:LED-SMD_4P-L1.6-W1.5_XL-1615RGBC-WS2812B, F.Cu at (169.1, 346.9)
- added D236: XL-1615RGBC-WS2812B-S, PCM_JLCPCB:LED-SMD_4P-L1.6-W1.5_XL-1615RGBC-WS2812B, F.Cu at (171.8, 349.0)
- added D237: XL-1615RGBC-WS2812B-S, PCM_JLCPCB:LED-SMD_4P-L1.6-W1.5_XL-1615RGBC-WS2812B, F.Cu at (210.6, -177.2)
- added D238: XL-1615RGBC-WS2812B-S, PCM_JLCPCB:LED-SMD_4P-L1.6-W1.5_XL-1615RGBC-WS2812B, F.Cu at (210.6, -174.5)
- added D239: XL-1615RGBC-WS2812B-S, PCM_JLCPCB:LED-SMD_4P-L1.6-W1.5_XL-1615RGBC-WS2812B, F.Cu at (210.6, -171.8)
- added D240: XL-1615RGBC-WS2812B-S, PCM_JLCPCB:LED-SMD_4P-L1.6-W1.5_XL-1615RGBC-WS2812B, F.Cu at (214.1, -206.3)
- added D241: XL-1615RGBC-WS2812B-S, PCM_JLCPCB:LED-SMD_4P-L1.6-W1.5_XL-1615RGBC-WS2812B, F.Cu at (214.1, -203.7)
- added D242: XL-1615RGBC-WS2812B-S, PCM_JLCPCB:LED-SMD_4P-L1.6-W1.5_XL-1615RGBC-WS2812B, F.Cu at (214.1, -201.0)
- added D243: XL-1615RGBC-WS2812B-S, PCM_JLCPCB:LED-SMD_4P-L1.6-W1.5_XL-1615RGBC-WS2812B, F.Cu at (214.1, -198.3)
- added D244: XL-1615RGBC-WS2812B-S, PCM_JLCPCB:LED-SMD_4P-L1.6-W1.5_XL-1615RGBC-WS2812B, F.Cu at (214.1, -195.7)
- added D245: XL-1615RGBC-WS2812B-S, PCM_JLCPCB:LED-SMD_4P-L1.6-W1.5_XL-1615RGBC-WS2812B, F.Cu at (214.1, -193.1)
- added D246: XL-1615RGBC-WS2812B-S, PCM_JLCPCB:LED-SMD_4P-L1.6-W1.5_XL-1615RGBC-WS2812B, F.Cu at (214.1, -190.4)
- added D247: XL-1615RGBC-WS2812B-S, PCM_JLCPCB:LED-SMD_4P-L1.6-W1.5_XL-1615RGBC-WS2812B, F.Cu at (214.1, -187.8)
- added D248: XL-1615RGBC-WS2812B-S, PCM_JLCPCB:LED-SMD_4P-L1.6-W1.5_XL-1615RGBC-WS2812B, F.Cu at (214.1, -185.1)
- added D249: XL-1615RGBC-WS2812B-S, PCM_JLCPCB:LED-SMD_4P-L1.6-W1.5_XL-1615RGBC-WS2812B, F.Cu at (214.1, -182.4)
- added D250: XL-1615RGBC-WS2812B-S, PCM_JLCPCB:LED-SMD_4P-L1.6-W1.5_XL-1615RGBC-WS2812B, F.Cu at (214.1, -179.8)
- added D251: XL-1615RGBC-WS2812B-S, PCM_JLCPCB:LED-SMD_4P-L1.6-W1.5_XL-1615RGBC-WS2812B, F.Cu at (214.1, -177.2)
- added D252: XL-1615RGBC-WS2812B-S, PCM_JLCPCB:LED-SMD_4P-L1.6-W1.5_XL-1615RGBC-WS2812B, F.Cu at (214.1, -174.5)
- added D253: XL-1615RGBC-WS2812B-S, PCM_JLCPCB:LED-SMD_4P-L1.6-W1.5_XL-1615RGBC-WS2812B, F.Cu at (214.1, -171.8)
- added D254: XL-1615RGBC-WS2812B-S, PCM_JLCPCB:LED-SMD_4P-L1.6-W1.5_XL-1615RGBC-WS2812B, F.Cu at (217.5, -206.3)
- added D255: XL-1615RGBC-WS2812B-S, PCM_JLCPCB:LED-SMD_4P-L1.6-W1.5_XL-1615RGBC-WS2812B, F.Cu at (217.5, -203.7)
- added D256: XL-1615RGBC-WS2812B-S, PCM_JLCPCB:LED-SMD_4P-L1.6-W1.5_XL-1615RGBC-WS2812B, F.Cu at (217.5, -201.0)
- added D257: XL-1615RGBC-WS2812B-S, PCM_JLCPCB:LED-SMD_4P-L1.6-W1.5_XL-1615RGBC-WS2812B, F.Cu at (217.5, -198.3)
- added D258: XL-1615RGBC-WS2812B-S, PCM_JLCPCB:LED-SMD_4P-L1.6-W1.5_XL-1615RGBC-WS2812B, F.Cu at (217.5, -195.7)
- added D259: XL-1615RGBC-WS2812B-S, PCM_JLCPCB:LED-SMD_4P-L1.6-W1.5_XL-1615RGBC-WS2812B, F.Cu at (217.5, -193.1)
- added D260: XL-1615RGBC-WS2812B-S, PCM_JLCPCB:LED-SMD_4P-L1.6-W1.5_XL-1615RGBC-WS2812B, F.Cu at (217.5, -190.4)
- added D261: XL-1615RGBC-WS2812B-S, PCM_JLCPCB:LED-SMD_4P-L1.6-W1.5_XL-1615RGBC-WS2812B, F.Cu at (217.5, -187.8)
- added D262: XL-1615RGBC-WS2812B-S, PCM_JLCPCB:LED-SMD_4P-L1.6-W1.5_XL-1615RGBC-WS2812B, F.Cu at (217.5, -185.1)
- added D263: XL-1615RGBC-WS2812B-S, PCM_JLCPCB:LED-SMD_4P-L1.6-W1.5_XL-1615RGBC-WS2812B, F.Cu at (217.5, -182.4)
- added D264: XL-1615RGBC-WS2812B-S, PCM_JLCPCB:LED-SMD_4P-L1.6-W1.5_XL-1615RGBC-WS2812B, F.Cu at (217.5, -179.8)
- added D265: XL-1615RGBC-WS2812B-S, PCM_JLCPCB:LED-SMD_4P-L1.6-W1.5_XL-1615RGBC-WS2812B, F.Cu at (217.5, -177.2)
- added D266: XL-1615RGBC-WS2812B-S, PCM_JLCPCB:LED-SMD_4P-L1.6-W1.5_XL-1615RGBC-WS2812B, F.Cu at (217.5, -174.5)
- added D4: MM1W5V6, PCM_JLCPCB:D_SOD-123, F.Cu at (105.5, 359.4)
- added D5: MM1W5V6, PCM_JLCPCB:D_SOD-123, F.Cu at (96.8, 359.6)
- added D8: Green, PCM_JLCPCB:D_0805, F.Cu at (87.4, 365.0)
- added D9: Green, PCM_JLCPCB:D_0805, F.Cu at (63.3, 365.0)
- added F1: Polyfuse, 2A, Fuse:Fuse_1206_3216Metric, F.Cu at (101.7, 361.0)
- added G***: LOGO, LOGO, F.Cu at (58.8, 364.0)
- added G***: LOGO, LOGO, B.Cu at (87.1, 363.8)
- added G***: LOGO, LOGO, B.Cu at (115.4, 364.1)
- added G***: LOGO, LOGO, B.Cu at (62.4, 364.1)
- added G***: LOGO, LOGO, B.Cu at (75.3, 364.0)
- added G***: LOGO, LOGO, B.Cu at (140.5, 356.0)
- added G***: LOGO, Custom_Footprints:Power, F.Cu at (82.9, 364.0)
- added G***: LOGO, Custom_Footprints:WiFi, F.Cu at (71.2, 364.0)
- added G***: LOGO, LOGO, F.Cu at (129.7, 164.8)
- added G***: LOGO, Custom_Footprints:Mode_Off_ON, F.Cu at (61.5, 234.0)
- added G***: LOGO, Custom_Footprints:Brightness_7, F.Cu at (61.5, 245.2)
- added G***: LOGO, LOGO, F.Cu at (61.6, 239.5)
- added G***: LOGO, Custom_Footprints:Brightness_0, F.Cu at (61.5, 250.8)
- added G***: LOGO, Custom_Footprints:Power, B.Cu at (137.5, 356.0)
- added J1: Prog Connector, Custom_Footprints:Prog Connector, F.Cu at (61.8, 319.8)
- added L1: 2.7nH, PCM_JLCPCB:L_0402, F.Cu at (59.2, 344.4)
- added L5: 15nH,300mA, PCM_JLCPCB:L_0402, F.Cu at (61.7, 341.9)
- added Q1: HL3415A, PCM_JLCPCB:Q_SOT-23, F.Cu at (101.2, 356.4)
- added Q2: MMBT3904, PCM_JLCPCB:Q_SOT-23, F.Cu at (97.3, 356.4)
- added R1: 10kΩ, PCM_JLCPCB:R_0402, F.Cu at (71.4, 344.1)
- added R12: 10kΩ, PCM_JLCPCB:R_0402, F.Cu at (89.9, 363.0)
- added R13: 5.1kΩ, PCM_JLCPCB:R_0402, F.Cu at (134.6, 360.6)
- added R14: 5.1kΩ, PCM_JLCPCB:R_0402, F.Cu at (134.6, 351.4)
- added R15: 510Ω, PCM_JLCPCB:R_0402, F.Cu at (75.0, 352.6)
- added R16: 100kΩ, PCM_JLCPCB:R_0402, F.Cu at (94.3, 354.9)
- added R17: 10kΩ, PCM_JLCPCB:R_0402, F.Cu at (94.3, 357.9)
- added R18: 510Ω, PCM_JLCPCB:R_0402, F.Cu at (94.3, 356.9)
- added R2: 10kΩ, PCM_JLCPCB:R_0402, F.Cu at (72.7, 345.3)
- added R21: 10kΩ, PCM_JLCPCB:R_0402, F.Cu at (78.2, 363.0)
- added R22: 100kΩ, PCM_JLCPCB:R_0402, F.Cu at (65.8, 365.0)
- added R23: 100kΩ, PCM_JLCPCB:R_0402, F.Cu at (78.2, 365.0)
- added R25: 100kΩ, PCM_JLCPCB:R_0402, F.Cu at (76.4, 353.3)
- added R3: 10kΩ, PCM_JLCPCB:R_0402, F.Cu at (67.4, 354.9)
- added R4: 5.1kΩ, PCM_JLCPCB:R_0402, F.Cu at (68.1, 354.2)
- added R5: 10kΩ, PCM_JLCPCB:R_0402, F.Cu at (69.5, 352.8)
- added R7: 510Ω, PCM_JLCPCB:R_0402, F.Cu at (63.2, 336.1)
- added R8: 10kΩ, PCM_JLCPCB:R_0402, F.Cu at (65.8, 363.0)
- added R9: 100kΩ, PCM_JLCPCB:R_0402, F.Cu at (89.9, 365.0)
- added REF**: MountingHole_3.2mm_M3, MountingHole:MountingHole_3.2mm_M3, F.Cu at (54.5, 364.0)
- added REF**: MountingHole_3.2mm_M3, MountingHole:MountingHole_3.2mm_M3, F.Cu at (138.5, 364.0)
- added S1: Tactile Button, 160gf, PCM_JLCPCB:SW-SMD_4P-L5.1-W5.1-P3.70-LS6.5-TL-2, F.Cu at (68.5, 234.0)
- added S2: Tactile Button, 160gf, PCM_JLCPCB:SW-SMD_4P-L5.1-W5.1-P3.70-LS6.5-TL-2, F.Cu at (68.5, 245.2)
- added S3: Tactile Button, 160gf, PCM_JLCPCB:SW-SMD_4P-L5.1-W5.1-P3.70-LS6.5-TL-2, F.Cu at (68.5, 250.8)
- added S4: Tactile Button, 160gf, PCM_JLCPCB:SW-SMD_4P-L5.1-W5.1-P3.70-LS6.5-TL-2, F.Cu at (68.5, 239.6)
- added U1: RT9080-33GJ5, Package_TO_SOT_SMD:TSOT-23-5, F.Cu at (63.0, 354.5)
- added U2: ESP32-C3FH4, PCM_JLCPCB:QFN-32-1EP_5x5mm_P0.5mm_EP3.7x3.7mm_ThermalVias, F.Cu at (65.0, 343.9)
- added U3: LTR-303ALS-01, PCM_JLCPCB:Lite-On_LTR-303ALS-01, F.Cu at (71.5, 356.3)
- added U4: Connector, USB-TYPE-C-16P, Custom_Footprints:TYPE-C-SMD_HX-TYPE-C-16PIN, F.Cu at (138.5, 356.0)
- added U5: SN74LV1T34DBV, Package_TO_SOT_SMD:SOT-23-5, F.Cu at (73.6, 349.8)
- added X1: 40MHz, 15pF, Custom_Footprints:OSC-SMD_4P-L3.2-W2.5-BL_SIT8008BI, F.Cu at (60.7, 339.2)
- added kibuzzard-68A93B9D: G***, kibuzzard-68A93B9D, B.Cu at (64.7, 319.8)
- added kibuzzard-68A93BAB: G***, kibuzzard-68A93BAB, B.Cu at (64.9, 322.3)
- added kibuzzard-68A93BBD: G***, kibuzzard-68A93BBD, B.Cu at (66.3, 324.9)
- added kibuzzard-68A93BCF: G***, kibuzzard-68A93BCF, B.Cu at (65.6, 327.4)
- added kibuzzard-68A93BEA: G***, kibuzzard-68A93BEA, B.Cu at (64.2, 330.0)
- added kibuzzard-68A93BF1: G***, kibuzzard-68A93BF1, B.Cu at (64.3, 332.5)
Routing:
- net VBUS: track 0.00 -> 127.0 mm, vias 0 -> 10
- net /D+: track 0.00 -> 112.9 mm, vias 0 -> 2
- net /D-: track 0.00 -> 109.0 mm, vias 0 -> 2
- net +3V3: track 0.00 -> 105.0 mm, vias 0 -> 20
- net /+BRIGHTNESS_BUTTON: track 0.00 -> 104.5 mm, vias 0 -> 7
- net Net-(C13-Pad1): track 0.00 -> 101.5 mm, vias 0 -> 6
- net /MODE_BUTTON: track 0.00 -> 96.2 mm, vias 0 -> 3
- net /BOOT_IO9_BUTTON: track 0.00 -> 95.6 mm, vias 0 -> 4
- net /-BRIGHTNESS_BUTTON: track 0.00 -> 77.3 mm, vias 0 -> 3
- net /Reset: track 0.00 -> 48.7 mm, vias 0 -> 6
- net GND: track 0.00 -> 44.3 mm, vias 0 -> 308
- net /SERVER_LED: track 0.00 -> 40.2 mm, vias 0 -> 2
- net /LED_POWER_ENABLE: track 0.00 -> 35.3 mm, vias 0 -> 4
- net LED_DATA_5V: track 0.00 -> 33.5 mm, vias 0 -> 2
- net /WIFI_LED: track 0.00 -> 29.3 mm, vias 0 -> 2
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- added copper zone on F.Cu, net +3V3
- added copper zone on F.Cu, net /Antenna
- added copper zone on F.Cu, net GND
Other:
- board outline added: 200 x 320 mm
- board text added: "Bridge Street"
- board text added: "Central Chalmers Street"
- board text added: "Chinatown"
- board text added: "Circular Quay"
- board text added: "Designed in Aotearoa, Made in Shenzhen"
- board text added: "ES Marks"
- board text added: "Haymarket"
- board text added: "Juniors Kingsford"
- board text added: "Kea Studios"
- board text added: "Kensington"
- board text added: "Kingsford"
- board text added: "Light Rail"
- board text added: "Moore Park"
- board text added: "Network"
- board text added: "Next departures to Circular Quay"
- board text added: "QVB"
- board text added: "REF**"
- board text added: "Randwick"
- board text added: "Royal Randwick"
- board text added: "Surry Hills"
- board text added: "Sydney"
- board text added: "Town Hall"
- board text added: "UNSW ANZAC Parade"
- board text added: "UNSW Anzac Parade"
- board text added: "UNSW High Street"
- board text added: "V1.0.0 08/2025"
- board text added: "Wansey Road"
- board text added: "Wynyard"
- board text added: "keastudios.co.nz/wlg-ltm-quick-start"

Commit message: Added Metro icon
Routing:
- added copper zone on F.Cu, net (none)
